File: Atmega328P/Atmega328P.kicad_sch (KiCad schematic)
At the start: 25 parts, among them U1 24LC1025, U2 DS1337S_, U3 24LC1025, U4 ATMEGA328P-AU, Y1 32.768 KHz, Y2 16 MHz

Commit message: SCL Error- solver in schematic.
Connections:
- net SCL: no longer D1.2 (A), U4.17 (PB5)
- new net SCK: D1.2 (A), U4.17 (PB5)
Other:
- sheet Connectors ports: added VCC; removed Vcc
- moved on the sheet: BT1, C1, C2, C3, C4, C5, D2, R1, R2, R3, R4, R5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
