File: Atmega328P/Connectors_Sheet.kicad_sch (KiCad schematic)
At the start: 4 parts, among them J1 Conn_01x04_Pin, J2 Conn_01x09_Pin, J3 Conn_01x04_Pin, J4 Conn_02x03_Odd_Even

Commit message: SCL Error- solver in schematic.
Connections:
- net Vcc renamed VCC
Other:
- moved on the sheet: J2, J3, J4
